File: pcb/R1007.kicad_pcb (KiCad board)
At the start: 2 copper layers, 45 x 33.3 mm, 1 part, among them J1 PCIEx1Edge

Commit message: wip, need to add 74 buffers and LEDs
Parts:
- added J2: CONN500P-01X04, Main:CONN500P-01X04, F.Cu at (130.0, 100.0)
- added J3: CONN_R1000A_EXTENSION, Main:CONN127P-02X10, F.Cu at (126.9, 80.0)
- added Q1: PSMN1R2-30YLC, Main:SOT127P500X110-5, F.Cu at (150.0, 75.0)
- added Q2: PSMN1R2-30YLC, Main:SOT127P500X110-5, F.Cu at (150.0, 85.0)
- added Q3: PSMN1R2-30YLC, Main:SOT127P500X110-5, F.Cu at (150.0, 95.0)
- added Q4: PSMN1R2-30YLC, Main:SOT127P500X110-5, F.Cu at (150.0, 105.0)
- added R1: 10k, Resistors_SMD:R_0603, F.Cu at (135.9, 70.4)
- added R10: 10k, Resistors_SMD:R_0603, F.Cu at (139.1, 70.4)
- added R11: 10k, Resistors_SMD:R_0603, F.Cu at (146.4, 109.0)
- added R12: 10k, Resistors_SMD:R_0603, F.Cu at (146.4, 99.0)
- added R13: 10k, Resistors_SMD:R_0603, F.Cu at (146.4, 89.0)
- added R14: 10k, Resistors_SMD:R_0603, F.Cu at (146.4, 79.0)
- added R2: 10k, Resistors_SMD:R_0603, F.Cu at (134.3, 70.4)
- added R3: 10k, Resistors_SMD:R_0603, F.Cu at (132.7, 70.4)
- added R4: 10k, Resistors_SMD:R_0603, F.Cu at (131.1, 70.4)
- added R5: 10k, Resistors_SMD:R_0603, F.Cu at (129.5, 70.4)
- added R6: 10k, Resistors_SMD:R_0603, F.Cu at (137.5, 70.4)
- added R7: 10k, Resistors_SMD:R_0603, F.Cu at (143.9, 70.4)
- added R8: 10k, Resistors_SMD:R_0603, F.Cu at (142.3, 70.4)
- added R9: 10k, Resistors_SMD:R_0603, F.Cu at (140.7, 70.4)
- added U2: AS78L05ZTR-E1, Main:TO92_AMMO, F.Cu at (138.7, 108.7)
- added U3: TLP293-4, Main:SOIC127P1030X455X210-16, F.Cu at (134.1, 79.6)
- J1: value PCIEx1Edge -> CONN500P-01X08; footprint Main:PCIEXPRESS-X1 -> Main:CONN500P-01X08; moved to F.Cu
- moved J1 15.6 mm to (162.0, 90.0), turned to 90 degrees
Routing:
- net Net-(J1-PadB9): track 2.30 -> 0.00 mm
- net Net-(J1-PadB8): track 2.30 -> 0.00 mm
- net Net-(J1-PadB7): track 2.30 -> 0.00 mm
- net Net-(J1-PadB6): track 2.30 -> 0.00 mm
- net Net-(J1-PadB5): track 2.30 -> 0.00 mm
- net Net-(J1-PadB4): track 2.30 -> 0.00 mm
- net Net-(J1-PadB3): track 2.30 -> 0.00 mm
- net Net-(J1-PadB2): track 2.30 -> 0.00 mm
- net Net-(J1-PadB18): track 2.30 -> 0.00 mm
- net Net-(J1-PadB16): track 2.30 -> 0.00 mm
- net Net-(J1-PadB15): track 2.30 -> 0.00 mm
- net Net-(J1-PadB14): track 2.30 -> 0.00 mm
- net Net-(J1-PadB13): track 2.30 -> 0.00 mm
- net Net-(J1-PadB12): track 2.30 -> 0.00 mm
- net Net-(J1-PadB11): track 2.30 -> 0.00 mm
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Other:
- board size 45 x 33.3 mm -> 52 x 44 mm
- copper layers 2 -> 4

Commit message: released first version
Parts:
- added C1: 1uF, Capacitors_SMD:C_0603, F.Cu at (132.9, 109.6)
- added C2: 1uF, Capacitors_SMD:C_0603, F.Cu at (132.9, 104.5)
- added D1: Led_Small, LEDs:LED_0805, F.Cu at (146.1, 79.1)
- added D2: Led_Small, LEDs:LED_0805, F.Cu at (146.1, 89.1)
- added D3: Led_Small, LEDs:LED_0805, F.Cu at (146.1, 99.1)
- added D4: Led_Small, LEDs:LED_0805, F.Cu at (146.1, 109.1)
- added G***: LOGO, pluggee:pluggee-QRNEG-127X127, F.Cu at (131.5, 92.5)
- added G***: LOGO, pluggee:pluggee-LOGO-131X127, B.Cu at (152.6, 80.7)
- added G***: LOGO, pluggee:pluggee-QRNEG-190X190, B.Cu at (142.0, 97.7)
- added MP1: MECH_NPTH_M3, Main:MECH_NPTH_M3, F.Cu at (169.0, 109.0)
- added MP2: MECH_NPTH_M3, Main:MECH_NPTH_M3, F.Cu at (169.0, 71.0)
- added MP3: MECH_NPTH_M3, Main:MECH_NPTH_M3, F.Cu at (106.0, 71.0)
- added MP4: MECH_NPTH_M3, Main:MECH_NPTH_M3, F.Cu at (106.0, 109.0)
- added R15: 1k, Resistors_SMD:R_0603, F.Cu at (142.6, 79.1)
- added R16: 1k, Resistors_SMD:R_0603, F.Cu at (142.6, 89.1)
- added R17: 1k, Resistors_SMD:R_0603, F.Cu at (142.6, 99.1)
- added R18: 1k, Resistors_SMD:R_0603, F.Cu at (142.6, 109.1)
- added U1: 74HC125, Main:SOIC127P870X390X175-14, F.Cu at (129.6, 72.9)
- R10, R7, R8, R9: value 10k -> 1k
- R11, R12, R13, R14: value 10k -> 4.7k
- moved R11 32.9 mm to (125.2, 83.9), turned to 0 degrees
- moved R12 27.1 mm to (125.2, 82.1), turned to 0 degrees
- moved R1 26.8 mm to (109.1, 70.5)
- moved R2 23.6 mm to (110.7, 70.5)
- moved R13 22.9 mm to (125.2, 80.3), turned to 0 degrees
- moved R14 21.2 mm to (125.2, 78.5), turned to 0 degrees
- moved R6 20.4 mm to (117.1, 70.5)
- moved R7 20.4 mm to (123.5, 70.5)
- moved R8 20.4 mm to (121.9, 70.5)
- moved R10 20.4 mm to (118.7, 70.5)
- moved R3 20.4 mm to (112.3, 70.5)
- moved R9 20.4 mm to (120.3, 70.5)
- moved R4 17.2 mm to (113.9, 70.5)
- moved J3 17.2 mm to (110.0, 83.0)
- moved U3 14.8 mm to (119.3, 79.4)
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Connections:
- J1 pad 1: Net-(J1-Pad1) -> /N4
- J1 pad 3: Net-(J1-Pad3) -> /N3
- J1 pad 5: Net-(J1-Pad5) -> /N2
- J1 pad 7: Net-(J1-Pad7) -> /N1
- Q1 pad 5: Net-(J1-Pad1) -> /N1
- Q2 pad 5: Net-(J1-Pad3) -> /N2
- Q3 pad 5: Net-(J1-Pad5) -> /N3
- Q4 pad 5: Net-(J1-Pad7) -> /N4
- R11 pad 1: /GN4 -> /IGN4
- R12 pad 1: /GN3 -> /IGN3
- R13 pad 1: /GN2 -> /IGN2
- R14 pad 1: /GN1 -> /IGN1
- U3 pad 11: /GN3 -> /IGN3
- U3 pad 13: /GN2 -> /IGN2
- U3 pad 15: /GN1 -> /IGN1
- U3 pad 9: /GN4 -> /IGN4
Routing:
- net /GN4: track 0.00 -> 52.9 mm, vias 0 -> 2
- net /GN3: track 0.00 -> 40.9 mm, vias 0 -> 2
- net ~MRESET: track 0.00 -> 36.9 mm, vias 0 -> 1
- net /GN2: track 0.00 -> 33.1 mm, vias 0 -> 2
- net /GN1: track 0.00 -> 31.0 mm, vias 0 -> 2
- net GND: track 0.00 -> 25.9 mm, vias 0 -> 1
- net C2D: track 0.00 -> 23.8 mm, vias 0 -> 1
- net +3V3: track 0.00 -> 21.3 mm, vias 0 -> 1
- net ID3: track 0.00 -> 21.1 mm, vias 0 -> 1
- net ID2: track 0.00 -> 20.6 mm, vias 0 -> 1
- net /IGN2: track 0.00 -> 20.4 mm, vias 0 -> 2
- net ID1: track 0.00 -> 19.6 mm, vias 0 -> 1
- net ID0: track 0.00 -> 18.9 mm, vias 0 -> 1
- net /INR4: track 0.00 -> 17.9 mm, vias 0 -> 2
- net +5P: track 0.00 -> 17.7 mm, vias 0 -> 2
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- added copper zone on In1.Cu, net +5P
- added copper zone on F.Cu, net /N1
- added copper zone on F.Cu, net /N2
- added copper zone on F.Cu, net /N3
- added copper zone on F.Cu, net /N4
- added copper zone on F.Cu, net GNDPWR
- added copper zone on B.Cu, net VDD
- added copper zone on In2.Cu, net VDD
Other:
- board size 52 x 44 mm -> 69 x 44 mm
- board text added: "+"
- board text added: "-"
- board text added: "1+"
- board text added: "1-"
- board text added: "2+"
- board text added: "2-"
- board text added: "3+"
- board text added: "3-"
- board text added: "4+"
- board text added: "4-"
- board text added: "HV In"
- board text added: "R1007 v1.0.0 Quad 20A NFET Drivers plugg.ee Labs 2016 http://plugg.ee"

Commit message: completed layout, wip
Parts:
- removed G***: LOGO, pluggee:pluggee-QRNEG-127X127
- removed G***: LOGO, pluggee:pluggee-LOGO-131X127
- removed G***: LOGO, pluggee:pluggee-QRNEG-190X190
- removed R1, R2, R3, R4, R5, R6: 10k, Resistors_SMD:R_0603
- added A1: ART, pluggee:pluggeeLabsIcon-13X7, B.Cu at (159.4, 87.0)
- added FID1: FIDTOP001, Main:FIDTOP001, F.Cu at (106.0, 99.6)
- added FID2: FIDTOP001, Main:FIDTOP001, F.Cu at (169.0, 99.6)
- added FID3: FIDTOP001, Main:FIDTOP001, F.Cu at (106.0, 75.0)
- C1, C2: value 1uF -> CC0603KRX7R9BB104; footprint Capacitors_SMD:C_0603 -> Main:CAPC0603
- D1, D2, D3, D4: value Led_Small -> LTW-170TK; footprint LEDs:LED_0805 -> Main:DIOC200X120X110
- J2: value CONN500P-01X04 -> CONN500P-01X08; footprint Main:CONN500P-01X04 -> Main:CONN500P-01X08
- R10, R15, R16, R17, R18, R7, R8, R9: value 1k -> RC0603FR-071KL; footprint Resistors_SMD:R_0603 -> Main:RESC0603
- R11, R12, R13, R14: value 4.7k -> RC0603FR-074K7L; footprint Resistors_SMD:R_0603 -> Main:RESC0603
- moved Q4 26.9 mm to (129.8, 87.3), turned to 0 degrees
- moved J2 26.5 mm to (144.8, 97.6), turned to 0 degrees
- moved R15 24.9 mm to (165.6, 88.6), turned to 270 degrees
- moved D4 24.2 mm to (133.9, 88.2), turned to 270 degrees
- moved R18 21.7 mm to (135.6, 88.6), turned to 270 degrees
- moved J1 21.6 mm to (144.8, 77.0), turned to 180 degrees
- moved D1 20.0 mm to (163.9, 88.2), turned to 270 degrees
- moved C2 19.6 mm to (115.8, 95.0), turned to 180 degrees
- moved C1 19.5 mm to (115.8, 100.2), turned to 180 degrees
- moved U1 17.9 mm to (119.6, 87.8), turned to 180 degrees
- moved Q1 15.7 mm to (159.8, 87.3), turned to 0 degrees
- moved R14 15.4 mm to (114.7, 89.7), turned to 270 degrees
- moved R16 13.0 mm to (155.6, 88.6), turned to 270 degrees
- moved Q3 12.8 mm to (139.8, 87.3), turned to 0 degrees
- moved U2 12.6 mm to (120.1, 97.6)
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Connections:
- J1 pad 1: /N4 -> /N1
- J1 pad 3: /N3 -> /N2
- J1 pad 5: /N2 -> /N3
- J1 pad 7: /N1 -> /N4
- J2 pad 3: GNDPWR -> VDD
- J2 pad 4: VDD -> GNDPWR
- J3 pad 1: ~MRESET -> (no net)
- J3 pad 10: ID2 -> (no net)
- J3 pad 12: ID1 -> (no net)
- J3 pad 14: ID0 -> (no net)
- J3 pad 16: +3V3 -> (no net)
- J3 pad 2: C2D -> (no net)
- J3 pad 8: ID3 -> (no net)
Routing:
- net GNDPWR: track 0.00 -> 55.9 mm, vias 0 -> 48
- net /GN4: track 52.9 -> 13.5 mm
- net ~MRESET: track 36.9 -> 0.00 mm, vias 1 -> 0
- net /GN1: track 31.0 -> 58.5 mm
- net C2D: track 23.8 -> 0.00 mm, vias 1 -> 0
- net +5P: track 17.7 -> 39.6 mm, vias 2 -> 1
- net +3V3: track 21.3 -> 0.00 mm, vias 1 -> 0
- net ID3: track 21.1 -> 0.00 mm, vias 1 -> 0
- net ID2: track 20.6 -> 0.00 mm, vias 1 -> 0
- net ID1: track 19.6 -> 0.00 mm, vias 1 -> 0
- net ID0: track 18.9 -> 0.00 mm, vias 1 -> 0
- net /INR4: track 17.9 -> 1.70 mm, vias 2 -> 0
- net /N2: track 0.00 -> 15.8 mm, vias 0 -> 12
- net /N1: track 0.00 -> 15.8 mm, vias 0 -> 12
- net /N4: track 2.20 -> 14.9 mm, vias 0 -> 12
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- added copper zone on In1.Cu, net /N1
- added copper zone on In1.Cu, net /N2
- added copper zone on In1.Cu, net /N3
- added copper zone on In1.Cu, net /N4
- added copper zone on In1.Cu, net GNDPWR
- removed copper zone on In1.Cu, net +5P
Other:
- board size 69 x 44 mm -> 69 x 38.6 mm
- board text added: "OUT"
- board text added: "R1007 v1.1 Quad 20A NFET Drivers plugg.ee Labs LLC http://plugg.ee"
- board text removed: "R1007 v1.0.0 Quad 20A NFET Drivers plugg.ee Labs 2016 http://plugg.ee"
